File: PCB/Schematics/XDF-001.kicad_sch (KiCad schematic)
At the start: 23 parts, among them J1 Conn_01x02_MountingPin, J2 Conn_01x03_MountingPin, J3 Conn_01x02_MountingPin, J4 Conn_01x02_MountingPin, U10 MPU-9250_simplficado, U6 ESP32-DEVKITC_simplificado, U7 NRF24L01_simplificado, U8 PCA9685BS, U9 NEO-6M-GPS_simplificado

Commit message: Updated BOM, PCB Files for include capacitors and connectors, added HUD Functions
Parts:
- removed C6: C_Polarized, Capacitor_THT:CP_Radial_D4.0mm_P2.00mm, symbol Device:C_Polarized
- added C6: C, Capacitor_THT:C_Disc_D3.0mm_W1.6mm_P2.50mm, symbol Device:C
- C1, C11, C3, C5, C7, C9: footprint Capacitor_THT:C_Disc_D5.0mm_W2.5mm_P5.00mm -> Capacitor_THT:C_Disc_D3.0mm_W1.6mm_P2.50mm
- C10, C4: footprint Capacitor_THT:CP_Radial_D5.0mm_P2.50mm -> Capacitor_THT:CP_Radial_D5.0mm_P2.00mm
- C2, C8: footprint Capacitor_THT:CP_Radial_D5.0mm_P2.50mm -> Capacitor_THT:CP_Radial_D6.3mm_P2.50mm
Connections:
- net +3.3V: now also C6.1
- net GND: now also C6.2
Other:
- moved on the sheet: C8
